File: ECE_299_ALARM/ECE_299_ALARM.kicad_pcb (KiCad board)
At the start: 2 copper layers, 60 x 50 mm, 20 parts, among them SW1 SW_Push_Dual, SW2 SW_Push_Dual, SW3 SW_Push_Dual, SW4 SW_Push_Dual, U1 RDA5807M_Module, U2 RPi_Pico_TH, U3 LM386

Commit message: small_adjustments
Parts:
- moved LS1 1.34 mm to (143.2, 88.5)
- moved R2 1.31 mm to (143.2, 94.2)
- moved C2 0.79 mm to (140.8, 82.8)
Routing:
- net GND: track 130.6 -> 133.1 mm
- net Net-(LS1-Pad2): track 4.11 -> 3.23 mm
- net Net-(C2-Pad2): track 6.41 -> 5.72 mm
Changed lines of the file:
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@@
 	(footprint "Connector_PinHeader_2.54mm:PinHeader_1x02_P2.54mm_Vertical"
 		(layer "F.Cu")
-		(at 142 88)
+		(at 143.25 88.475)
 		(descr "Through hole straight pin header, 1x02, 2.54mm pitch, single row")
 		(tags "Through hole pin header THT 1x02 2.54mm single row")
 		(property "Reference" "LS1"
-			(at -3 0.5 0)
+			(at -3 -0.975 0)
 			(layer "F.SilkS")
 			(effects
@@
 		)
 		(property "Value" "Speaker"
-			(at 0 4.92 0)
+			(at 3.75 1.525 90)
 			(layer "F.Fab")
 			(effects
@@
 		)
 		(fp_text user "${REFERENCE}"
-			(at 0 1.27 90)
+			(at -3 -0.95 180)
 			(layer "F.Fab")
 			(effects
@@
 	(footprint "Resistor_THT:R_Axial_DIN0309_L9.0mm_D3.2mm_P12.70mm_Horizontal"
 		(layer "F.Cu")
-		(at 142 94.65 -90)
+		(at 143.25 94.25 -90)
 		(descr "Resistor, Axial_DIN0309 series, Axial, Horizontal, pin pitch=12.7mm, 0.5W = 1/2W, length*diameter=9*3.2mm^2, http://cdn-reichelt.de/documents/datenblatt/B400/1_4W%23YAG.pdf")
 		(tags "Resistor Axial_DIN0309 series Axial Horizontal pin pitch 12.7mm 0.5W = 1/2W length 9mm diameter 3.2mm")
 		(property "Reference" "R2"
-			(at 6.35 0 90)
+			(at 6.35 0 180)
 			(layer "F.SilkS")
 			(effects
@@
 		(tags "C Radial series Radial pin pitch 2.50mm diameter 6.3mm height 11mm Non-Polar Electrolytic Capacitor")
 		(property "Reference" "C1"
-			(at 4 -3.5 0)
+			(at 1.25 -1.5 0)
 			(layer "F.SilkS")
 			(effects
@@
 		(at 108 78 90)
 		(property "Reference" "U1"
-			(at 0 -3.5 0)
+			(at 0 0 0)
 			(unlocked yes)
 			(layer "F.SilkS")
@@
 	(footprint "Capacitor_THT:C_Radial_D6.3mm_H11.0mm_P2.50mm"
 		(layer "F.Cu")
-		(at 140.5 82)
+		(at 140.75 82.75)
 		(descr "C, Radial series, Radial, pin pitch=2.50mm, diameter=6.3mm, height=11mm, Non-Polar Electrolytic Capacitor")
 		(tags "C Radial series Radial pin pitch 2.50mm diameter 6.3mm height 11mm Non-Polar Electrolytic Capacitor")
@@
 		(at 113 100 90)
 		(property "Reference" "U2"
-			(at 0 0 90)
+			(at 0 0 0)
 			(unlocked yes)
 			(layer "F.SilkS")
@@
 		)
 		(property "Value" "RPi_Pico_TH"
-			(at 0 2.54 90)
+			(at 0 6.75 0)
 			(unlocked yes)
 			(layer "F.Fab")
@@
 		)
 		(fp_text user "${REFERENCE}"
-			(at 0 -2.54 90)
+			(at -1.75 -0.75 0)
 			(unlocked yes)
 			(layer "F.Fab")
@@
 	)
 	(segment
-		(start 143 87)
-		(end 142 88)
+		(start 143.25 82.75)
+		(end 143.25 88.475)
 		(width 1)
 		(layer "F.Cu")
@@
 	)
 	(segment
-		(start 143 82)
-		(end 143 87)
-		(width 1)
-		(layer "F.Cu")
-		(net 4)
-	)
-	(segment
-		(start 139.69 82.81)
-		(end 140.5 82)
+		(start 135.815 82.81)
+		(end 135.875 82.75)
 		(width 1)
 		(layer "F.Cu")
@@
 	)
 	(segment
-		(start 135.815 82.81)
-		(end 139.69 82.81)
+		(start 135.875 82.75)
+		(end 140.75 82.75)
 		(width 1)
 		(layer "F.Cu")
@@
 	)
 	(segment
-		(start 136.6 112.75)
-		(end 133.5 112.75)
-		(width 0.2)
-		(layer "F.Cu")
-		(net 6)
-	)
-	(segment
 		(start 112 72.6)
 		(end 113.1 71.5)
@@
 	)
 	(segment
-		(start 142 107.35)
-		(end 136.6 112.75)
+		(start 133.5 112.75)
+		(end 137.45 112.75)
+		(width 0.2)
+		(layer "F.Cu")
+		(net 6)
+	)
+	(segment
+		(start 137.45 112.75)
+		(end 143.25 106.95)
 		(width 0.2)
 		(layer "F.Cu")
@@
 	)
 	(segment
+		(start 138.25 88.75)
+		(end 140.25 90.75)
+		(width 1)
+		(layer "B.Cu")
+		(net 6)
+	)
+	(segment
 		(start 106.727156 112.772844)
 		(end 106.75 112.75)
@@
 	)
 	(segment
-		(start 133.66 89.5)
-		(end 137.75 89.5)
-		(width 1)
+		(start 132.16 86.5)
+		(end 134.41 88.75)
+		(width 0.2)
 		(layer "B.Cu")
 		(net 6)
@@
 	)
 	(segment
-		(start 137.75 89.5)
-		(end 139.5 91.25)
+		(start 140.25 90.75)
+		(end 140.25 103.95)
 		(width 1)
 		(layer "B.Cu")
@@
 	)
 	(segment
+		(start 132 86.5)
+		(end 132.16 86.5)
+		(width 0.2)
+		(layer "B.Cu")
+		(net 6)
+	)
+	(segment
 		(start 116.75 112.75)
 		(end 123.25 112.75)
@@
 	)
 	(segment
+		(start 133.66 89.5)
+		(end 134.41 88.75)
+		(width 1)
+		(layer "B.Cu")
+		(net 6)
+	)
+	(segment
+		(start 134.41 88.75)
+		(end 138.25 88.75)
+		(width 1)
+		(layer "B.Cu")
+		(net 6)
+	)
+	(segment
 		(start 128.195 77.73)
 		(end 129.296 78.831)
@@
 	)
 	(segment
-		(start 132 86.5)
-		(end 133.66 88.16)
-		(width 0.2)
-		(layer "B.Cu")
-		(net 6)
-	)
-	(segment
 		(start 132.05 91.11)
 		(end 133.66 89.5)
@@
 	)
 	(segment
-		(start 139.5 91.25)
-		(end 139.5 104.85)
+		(start 140.25 103.95)
+		(end 143.25 106.95)
 		(width 1)
 		(layer "B.Cu")
@@
 	)
 	(segment
-		(start 133.66 88.16)
-		(end 133.66 89.5)
-		(width 0.2)
-		(layer "B.Cu")
-		(net 6)
-	)
-	(segment
 		(start 96.80795 111.74795)
 		(end 96.80795 112.772844)
@@
 	)
 	(segment
-		(start 139.5 104.85)
-		(end 142 107.35)
-		(width 1)
-		(layer "B.Cu")
-		(net 6)
-	)
-	(segment
 		(start 118.8 74.5)
 		(end 115.8 71.5)
@@
 	)
 	(segment
-		(start 142 90.54)
-		(end 142 94.65)
+		(start 143.25 91.015)
+		(end 143.25 94.25)
 		(width 1)
 		(layer "F.Cu")
@@
 	)
 	(segment
-		(start 100.7 79.5)
-		(end 104 82.8)
-		(width 0.2)
-		(layer "F.Cu")
-		(net 15)
-	)
-	(segment
 		(start 103.9 83.5)
 		(end 104 83.4)
@@
 		(width 0.2)
 		(layer "B.Cu")
+		(net 15)
+	)
+	(segment
+		(start 102.5 83.5)
+		(end 102.5 83)
+		(width 0.2)
+		(layer "B.Cu")
+		(net 15)
+	)
+	(segment
+		(start 100.7 81.2)
+		(end 100.7 79.5)
+		(width 0.2)
+		(layer "B.Cu")
+		(net 15)
+	)
+	(segment
+		(start 102.5 83)
+		(end 100.7 81.2)
+		(width 0.2)
+		(layer "B.Cu")

Commit message: realized i also need to make the power supply lines wider too...
Parts:
- moved C1 0.25 mm to (119.5, 80.2)
Routing:
- net +5V: track 57.6 -> 65.8 mm, vias 4 -> 2
- net Net-(U3-+): track 17.0 -> 18.4 mm
- net GND: track 133.1 -> 133.8 mm
